Commit message: change optical flow axis
オプティカルフローセンサの座標軸の修正 #20
change optical flow axis, to Z-forward, X-right, Y-down

File: px4_gazebo_sim/urdf/adrien.urdf (robot description, URDF)
Before this commit: robot adrien, 28 links, 27 joints
Joints:
- joint optical_flow_bottom_joint: origin xyz=0.10783 -0.00735 -0.047658 rpy=-1.570796 1.570796 0 -> xyz=0.10783 -0.00735 -0.047658 rpy=-3.141593 0 0
- joint optical_flow_left_joint: origin xyz=-0.0077 0.048 -0.0672 rpy=0 0 1.570796 -> xyz=-0.0077 0.048 -0.0672 rpy=-1.570796 0 0
- joint optical_flow_right_joint: origin xyz=-0.0077 -0.048 -0.0672 rpy=0 0 -1.570796 -> xyz=-0.0077 -0.048 -0.0672 rpy=-1.570796 0 3.141593

Commit message: fix half of pi constant value
オプティカルフローセンサの座標軸の修正 #20

File: px4_gazebo_sim/urdf/adrien.urdf (robot description, URDF)
Before this commit: robot adrien, 28 links, 27 joints
Joints:
- joint camera_color_optical_joint: origin xyz=0 0 0  rpy=-1.57 0 -1.57 -> xyz=0 0 0  rpy=-1.570796 0 -1.570796
- joint camera_depth_optical_joint: origin xyz=0 0 0  rpy=-1.57 0 -1.57 -> xyz=0 0 0  rpy=-1.570796 0 -1.570796
- joint camera_left_ir_optical_joint: origin xyz=0 0 0  rpy=-1.57 0 -1.57 -> xyz=0 0 0  rpy=-1.570796 0 -1.570796
- joint camera_right_ir_optical_joint: origin xyz=0 0 0  rpy=-1.57 0 -1.57 -> xyz=0 0 0  rpy=-1.570796 0 -1.570796

Commit message: fix multizone lidar coordinate

File: px4_gazebo_sim/urdf/adrien.urdf (robot description, URDF)
Before this commit: robot adrien, 28 links, 27 joints
Joints:
- joint multi_zone_lidar_left_joint: origin xyz=0.0075 0.0465 -0.0665 rpy=0 0 1.570796 -> xyz=0.0075 0.0465 -0.0665 rpy=-1.570796 0 1.570796
- joint multi_zone_lidar_right_joint: origin xyz=0.0075 -0.0465 -0.0665 rpy=0 0 -1.570796 -> xyz=0.0075 -0.0465 -0.0665 rpy=1.570796 0 -1.570796

Commit message: fix imu frame

File: px4_gazebo_sim/urdf/adrien.urdf (robot description, URDF)
Before this commit: robot adrien, 28 links, 27 joints
Joints:
- joint imu_joint: origin xyz=0 0 0 rpy=0 0 0 -> xyz=0 0 0.025 rpy=3.141593 0 0

Commit message: fix rotation

File: px4_gazebo_sim/urdf/adrien.urdf (robot description, URDF)
Before this commit: robot adrien, 28 links, 27 joints
Links:
- added link optical_flow_top_link
Joints:
- added joint optical_flow_top_joint: type fixed, parent base_link, child optical_flow_top_link, origin xyz=0.0693 -0.00055 0.017 rpy=0 0 0

Commit message: add 上下のマルチゾーンLiDAR

File: px4_gazebo_sim/urdf/adrien.urdf (robot description, URDF)
Before this commit: robot adrien, 29 links, 28 joints
Links:
- added link multi_zone_lidar_bottom_link
- added link multi_zone_lidar_top_link
Joints:
- added joint multi_zone_lidar_bottom_joint: type fixed, parent base_link, child multi_zone_lidar_bottom_link, origin xyz=0.0875 0 -0.0555 rpy=0 1.570796 0
- added joint multi_zone_lidar_top_joint: type fixed, parent base_link, child multi_zone_lidar_top_link, origin xyz=0.0875 0 0.026 rpy=0 -1.570796 0
