Commit message: fix lidar roll value

File: adrien_driver/urdf/adrien.urdf (robot description, URDF)
Before this commit: robot adrien, 29 links, 28 joints
Joints:
- joint multi_zone_lidar_front_left_joint: origin xyz=0.113251 0.155545 -0.024 rpy=0 0 1.17809725 -> xyz=0.113251 0.155545 -0.024 rpy=1.570796 0 1.17809725
- joint multi_zone_lidar_front_right_joint: origin xyz=0.113251 -0.155545 -0.024 rpy=0 0 -1.17809725 -> xyz=0.113251 -0.155545 -0.024 rpy=1.570796 0 -1.17809725
- joint multi_zone_lidar_rear_left_joint: origin xyz=-0.113251 0.155545 -0.024 rpy=0 0 1.9634954 -> xyz=-0.113251 0.155545 -0.024 rpy=1.570796 0 1.9634954
- joint multi_zone_lidar_rear_right_joint: origin xyz=-0.113251 -0.155545 -0.024 rpy=0 0 -1.9634954 -> xyz=-0.113251 -0.155545 -0.024 rpy=1.570796 0 -1.9634954

Commit message: fix joint poses

File: adrien_driver/urdf/adrien.urdf (robot description, URDF)
Before this commit: robot adrien, 29 links, 28 joints
Joints:
- joint multi_zone_lidar_bottom_joint: origin xyz=0.1185 -0.0075 -0.0515 rpy=0 1.570796 0 -> xyz=0.1185 -0.0075 -0.0515 rpy=-1.570796 1.570796 0
- joint multi_zone_lidar_front_left_joint: origin xyz=0.113251 0.155545 -0.024 rpy=1.570796 0 1.17809725 -> xyz=0.113251 0.155545 -0.024 rpy=3.141593 0 1.17809725
- joint multi_zone_lidar_front_right_joint: origin xyz=0.113251 -0.155545 -0.024 rpy=1.570796 0 -1.17809725 -> xyz=0.113251 -0.155545 -0.024 rpy=3.141593 0 -1.17809725
- joint multi_zone_lidar_left_joint: origin xyz=-0.0075 0.0515 -0.0665 rpy=-1.570796 0 1.570796 -> xyz=-0.0075 0.0515 -0.0665 rpy=1.570796 0 1.570796
- joint multi_zone_lidar_rear_left_joint: origin xyz=-0.113251 0.155545 -0.024 rpy=1.570796 0 1.9634954 -> xyz=-0.113251 0.155545 -0.024 rpy=3.141593 0 1.9634954
- joint multi_zone_lidar_rear_right_joint: origin xyz=-0.113251 -0.155545 -0.024 rpy=1.570796 0 -1.9634954 -> xyz=-0.113251 -0.155545 -0.024 rpy=3.141593 0 -1.9634954
- joint multi_zone_lidar_right_joint: origin xyz=-0.0075 -0.0515 -0.0665 rpy=1.570796 0 -1.570796 -> xyz=-0.0075 -0.0515 -0.0665 rpy=-1.570796 0 -1.570796
- joint multi_zone_lidar_top_joint: origin xyz=0.0175 0.0075 0.0525 rpy=0 -1.570796 0 -> xyz=0.0175 0.0075 0.0525 rpy=1.570796 -1.570796 0
- joint optical_flow_bottom_joint: origin xyz=0.1178 -0.0077 -0.053 rpy=-3.141593 0 0 -> xyz=0.1178 -0.0077 -0.053 rpy=0 3.141593 0
- joint optical_flow_left_joint: origin xyz=-0.0077 0.055 -0.0672 rpy=-1.570796 0 0 -> xyz=-0.0077 0.055 -0.0672 rpy=0 -1.570796 -1.570796
- joint optical_flow_right_joint: origin xyz=-0.0077 -0.055 -0.0672 rpy=-1.570796 0 3.141593 -> xyz=-0.0077 -0.055 -0.0672 rpy=0 1.570796 -1.570796
- joint optical_flow_top_joint: origin xyz=0.0168 -0.0077 0.053 rpy=0 0 0 -> xyz=0.0168 -0.0077 0.053 rpy=0 0 3.141593
